Commit message: Wheels to My Robot

File: src/my_robot/urdf/my_robot.xacro (robot description, xacro)
@@ -7,4 +7,5 @@
     <child link="chassis" />
   </joint>
+  <!-- Chassis ======================================================= -->
   <link name='chassis'>
     <pose>0 0 0.1 0 0 0</pose>
@@ -55,3 +56,67 @@
     </visual>
   </link>
+  <!-- Wheels ======================================================= -->
+  <link name="left_wheel">
+    <!-- <pose>0 0 0.1 0 0 0</pose> -->
+    <inertial>
+      <mass value="5.0"/>
+      <origin xyz="0.0 0 0" rpy="0 1.5707 1.5707"/>
+      <inertia
+          ixx="0.1" ixy="0"   ixz="0"
+                    iyy="0.1" iyz="0"
+                              izz="0.1"
+      />
+    </inertial>
+    <collision name='left_wheel_collision'>
+      <origin xyz="0 0 0" rpy="0 1.5707 1.5707"/>
+      <geometry>
+        <cylinder radius="0.1" length="0.05"/>
+      </geometry>
+    </collision>
+    <visual name='left_wheel_visual'>
+      <origin xyz="0 0 0" rpy="0 1.5707 1.5707"/>
+      <geometry>
+        <cylinder radius="0.1" length="0.05"/>
+      </geometry>
+    </visual>
+  </link>
+  <link name="right_wheel">
+    <inertial>
+      <mass value="5.0"/>
+      <origin xyz="0.0 0 0" rpy="0 1.5707 1.5707"/>
+      <inertia
+          ixx="0.1" ixy="0"   ixz="0"
+                    iyy="0.1" iyz="0"
+                              izz="0.1"
+      />
+    </inertial>
+    <collision name='right_wheel_collision'>
+      <origin xyz="0 0 0" rpy="0 1.5707 1.5707"/>
+      <geometry>
+        <cylinder radius="0.1" length="0.05"/>
+      </geometry>
+    </collision>
+    <visual name='right_wheel_visual'>
+      <origin xyz="0 0 0" rpy="0 1.5707 1.5707"/>
+      <geometry>
+        <cylinder radius="0.1" length="0.05"/>
+      </geometry>
+    </visual>
+  </link>
+  <joint type="continuous" name="left_wheel_hinge">
+    <origin xyz="0 0.15 0" rpy="0 0 0"/>
+    <child link="left_wheel"/>
+    <parent link="chassis"/>
+    <axis xyz="0 1 0" rpy="0 0 0"/>
+    <limit effort="10000" velocity="1000"/>
+    <dynamics damping="1.0" friction="1.0"/>
+  </joint>
+  <joint type="continuous" name="right_wheel_hinge">
+    <origin xyz="0 -0.15 0" rpy="0 0 0"/>
+    <child link="right_wheel"/>
+    <parent link="chassis"/>
+    <axis xyz="0 -1 0" rpy="0 0 0"/>
+    <limit effort="10000" velocity="1000"/>
+    <dynamics damping="1.0" friction="1.0"/>
+  </joint>
 </robot>

Commit message: Add Sensors and Colors to MyRobot

File: src/my_robot/urdf/my_robot.xacro (robot description, xacro)
@@ -1,4 +1,17 @@
 <?xml version='1.0'?>
 <robot name="my_robot" xmlns:xacro="http://www.ros.org/wiki/xacro">
+<!-- I saw it done like this once, but it didn't work for me :/ - wrong file type :?
+  <material name="blue">
+    <color rgba="0 0 1 1"/>
+  </material>
+  <material name="black">
+    <color rgba="0 0 0 1"/>
+  </material>
+  <material name="red">
+    <color rgba="1 0 0 1"/>
+  </material>
+  <material name="green">
+    <color rgba="0 1 0 1"/>
+  </material> -->
   <link name="robot_footprint"></link>
   <joint name="robot_footprint_joint" type="fixed">
@@ -30,4 +43,5 @@
         <box size=".4 .2 .1"/>
       </geometry>
+      <!-- <material name="blue"/> -->
     </visual>
     <collision name='back_caster_collision'>
@@ -56,4 +70,7 @@
     </visual>
   </link>
+  <gazebo reference="chassis">
+      <material>Gazebo/Blue</material>
+  </gazebo>
   <!-- Wheels ======================================================= -->
   <link name="left_wheel">
@@ -79,6 +96,10 @@
         <cylinder radius="0.1" length="0.05"/>
       </geometry>
-    </visual>
-  </link>
+      <!-- <material name="green"/> -->
+    </visual>
+  </link>
+  <gazebo reference="left_wheel">
+      <material>Gazebo/Green</material>
+  </gazebo>
   <link name="right_wheel">
     <inertial>
@@ -102,6 +123,10 @@
         <cylinder radius="0.1" length="0.05"/>
       </geometry>
-    </visual>
-  </link>
+      <!-- <material name="green"/> -->
+    </visual>
+  </link>
+  <gazebo reference="right_wheel">
+      <material>Gazebo/Green</material>
+  </gazebo>
   <joint type="continuous" name="left_wheel_hinge">
     <origin xyz="0 0.15 0" rpy="0 0 0"/>
@@ -120,3 +145,69 @@
     <dynamics damping="1.0" friction="1.0"/>
   </joint>
+  <!-- Sensors ======================================================== -->
+  <link name="camera">
+    <inertial>
+      <mass value="0.1"/>
+      <origin xyz="0 0 0" rpy="0 0 0"/>
+      <inertia
+          ixx="1e-6" ixy="0"   ixz="0"
+                    iyy="1e-6" iyz="0"
+                              izz="1e-6"
+      />
+      <box_inertia m="0.1" x="0.05" y="0.05" z="0.05" />
+    </inertial>
+    <collision name='camera_collision'>
+      <origin xyz="0 0 0" rpy="0 0 0"/>
+      <geometry>
+        <box size="0.05 0.05 0.05"/>
+      </geometry>
+    </collision>
+    <visual name='camera_visual'>
+      <origin xyz="0 0 0" rpy="0 0 0"/>
+      <geometry>
+        <box size="0.05 0.05 0.05"/>
+      </geometry>
+      <!-- <material name="red"/> -->
+    </visual>
+  </link>
+  <gazebo reference="camera">
+      <material>Gazebo/Red</material>
+  </gazebo>
+  <joint type="fixed" name="camera_joint">
+    <origin xyz="0.2 0 0" rpy="0 0 0"/>
+    <child link="camera"/>
+    <parent link="chassis"/>
+    <axis xyz="0 1 0" rpy="0 0 0"/>
+  </joint>
+  <!-- Lidar  -->
+  <link name="hokuyo">
+    <inertial>
+      <mass value="1e-5"/>
+      <origin xyz="0 0 0" rpy="0 0 0"/>
+      <inertia
+          ixx="1e-6" ixy="0"   ixz="0"
+                    iyy="1e-6" iyz="0"
+                              izz="1e-6"
+      />
+      <!-- <box_inertia m="0.1" x="0.05" y="0.05" z="0.05" /> -->
+    </inertial>
+    <collision name='hokuyo_collision'>
+      <origin xyz="0 0 0" rpy="0 0 0"/>
+      <geometry>
+        <box size="0.1 0.1 0.1"/>
+      </geometry>
+    </collision>
+    <visual name='hokuyo_visual'>
+      <origin xyz="0 0 0" rpy="0 0 0"/>
+      <geometry >
+        <mesh filename="package://my_robot/meshes/hokuyo.dae"/>
+      </geometry>
+    </visual>
+  </link>
+  <joint type="fixed" name="hokuyo_joint">
+    <origin xyz="0.15 0 0.1" rpy="0 0 0"/>
+    <child link="hokuyo"/>
+    <parent link="chassis"/>
+    <axis xyz="0 1 0" rpy="0 0 0"/>
+  </joint>
 </robot>

Commit message: Update colors - to differenciate

File: src/my_robot/urdf/my_robot.xacro (robot description, xacro)
@@ -72,5 +72,5 @@
   </link>
   <gazebo reference="chassis">
-      <material>Gazebo/Blue</material>
+      <material>Gazebo/Green</material>
   </gazebo>
   <!-- Wheels ======================================================= -->
@@ -101,5 +101,5 @@
   </link>
   <gazebo reference="left_wheel">
-      <material>Gazebo/Green</material>
+      <material>Gazebo/Red</material>
   </gazebo>
   <link name="right_wheel">
@@ -128,5 +128,5 @@
   </link>
   <gazebo reference="right_wheel">
-      <material>Gazebo/Green</material>
+      <material>Gazebo/Red</material>
   </gazebo>
   <joint type="continuous" name="left_wheel_hinge">
@@ -173,5 +173,5 @@
   </link>
   <gazebo reference="camera">
-      <material>Gazebo/Red</material>
+      <material>Gazebo/Orange</material>
   </gazebo>
   <joint type="fixed" name="camera_joint">

Commit message: Scale the robot up a bit

File: src/my_robot/urdf/my_robot.xacro (robot description, xacro)
@@ -36,5 +36,5 @@
       <origin xyz="0 0 0" rpy=" 0 0 0"/>
       <geometry>
-        <box size=".4 .2 .1"/>
+        <box size=".8 .4 .1"/>
       </geometry>
     </collision>
@@ -42,30 +42,30 @@
       <origin xyz="0 0 0" rpy=" 0 0 0"/>
       <geometry>
-        <box size=".4 .2 .1"/>
+        <box size=".8 .4 .1"/>
       </geometry>
       <!-- <material name="blue"/> -->
     </visual>
     <collision name='back_caster_collision'>
-      <origin xyz="-0.15 0 -0.05" rpy=" 0 0 0"/>
-      <geometry>
-        <sphere radius="0.0499"/>
+      <origin xyz="-0.3 0 -0.075" rpy=" 0 0 0"/>
+      <geometry>
+        <sphere radius="0.07499"/>
       </geometry>
     </collision>
     <visual name='back_caster_visual'>
-      <origin xyz="-0.15 0 -0.05" rpy=" 0 0 0"/>
-      <geometry>
-        <sphere radius="0.05"/>
+      <origin xyz="-0.3 0 -0.075" rpy=" 0 0 0"/>
+      <geometry>
+        <sphere radius="0.075"/>
       </geometry>
     </visual>
     <collision name='front_caster_collision'>
-      <origin xyz="0.15 0 -0.05" rpy=" 0 0 0"/>
-      <geometry>
-        <sphere radius="0.0499"/>
+      <origin xyz="0.3 0 -0.075" rpy=" 0 0 0"/>
+      <geometry>
+        <sphere radius="0.07499"/>
       </geometry>
     </collision>
     <visual name='front_caster_visual'>
-      <origin xyz="0.15 0 -0.05" rpy=" 0 0 0"/>
-      <geometry>
-        <sphere radius="0.05"/>
+      <origin xyz="0.3 0 -0.075" rpy=" 0 0 0"/>
+      <geometry>
+        <sphere radius="0.075"/>
       </geometry>
     </visual>
@@ -87,13 +87,13 @@
     </inertial>
     <collision name='left_wheel_collision'>
-      <origin xyz="0 0 0" rpy="0 1.5707 1.5707"/>
-      <geometry>
-        <cylinder radius="0.1" length="0.05"/>
+      <origin xyz="0 0.1 0" rpy="0 1.5707 1.5707"/>
+      <geometry>
+        <cylinder radius="0.15" length="0.06"/>
       </geometry>
     </collision>
     <visual name='left_wheel_visual'>
-      <origin xyz="0 0 0" rpy="0 1.5707 1.5707"/>
-      <geometry>
-        <cylinder radius="0.1" length="0.05"/>
+      <origin xyz="0 0.1 0" rpy="0 1.5707 1.5707"/>
+      <geometry>
+        <cylinder radius="0.15" length="0.06"/>
       </geometry>
       <!-- <material name="green"/> -->
@@ -114,13 +114,13 @@
     </inertial>
     <collision name='right_wheel_collision'>
-      <origin xyz="0 0 0" rpy="0 1.5707 1.5707"/>
-      <geometry>
-        <cylinder radius="0.1" length="0.05"/>
+      <origin xyz="0 -0.1 0" rpy="0 1.5707 1.5707"/>
+      <geometry>
+        <cylinder radius="0.15" length="0.06"/>
       </geometry>
     </collision>
     <visual name='right_wheel_visual'>
-      <origin xyz="0 0 0" rpy="0 1.5707 1.5707"/>
-      <geometry>
-        <cylinder radius="0.1" length="0.05"/>
+      <origin xyz="0 -0.1 0" rpy="0 1.5707 1.5707"/>
+      <geometry>
+        <cylinder radius="0.15" length="0.06"/>
       </geometry>
       <!-- <material name="green"/> -->
@@ -150,5 +150,5 @@
     <inertial>
       <mass value="0.1"/>
-      <origin xyz="0 0 0" rpy="0 0 0"/>
+      <origin xyz="0.2 0 0" rpy="0 0 0"/>
       <inertia
           ixx="1e-6" ixy="0"   ixz="0"
@@ -159,5 +159,5 @@
     </inertial>
     <collision name='camera_collision'>
-      <origin xyz="0 0 0" rpy="0 0 0"/>
+      <origin xyz="0.2 0 0" rpy="0 0 0"/>
       <geometry>
         <box size="0.05 0.05 0.05"/>
@@ -165,5 +165,5 @@
     </collision>
     <visual name='camera_visual'>
-      <origin xyz="0 0 0" rpy="0 0 0"/>
+      <origin xyz="0.2 0 0" rpy="0 0 0"/>
       <geometry>
         <box size="0.05 0.05 0.05"/>

Commit message: Make the robot great again
The camera is round & black - as cameras tend to be
Also plugin is moved and wheels are not THAT sucky of
a collor

File: src/my_robot/urdf/my_robot.xacro (robot description, xacro)
@@ -101,5 +101,5 @@
   </link>
   <gazebo reference="left_wheel">
-      <material>Gazebo/Red</material>
+      <material>Gazebo/Orange</material>
   </gazebo>
   <link name="right_wheel">
@@ -128,5 +128,5 @@
   </link>
   <gazebo reference="right_wheel">
-      <material>Gazebo/Red</material>
+      <material>Gazebo/Orange</material>
   </gazebo>
   <joint type="continuous" name="left_wheel_hinge">
@@ -159,13 +159,15 @@
     </inertial>
     <collision name='camera_collision'>
-      <origin xyz="0.2 0 0" rpy="0 0 0"/>
-      <geometry>
-        <box size="0.05 0.05 0.05"/>
+      <origin xyz="0.2 0 0" rpy="0 1.5707 0"/>
+      <geometry>
+        <!-- <box size="0.05 0.05 0.05"/> -->
+        <cylinder radius="0.03" length="0.06"/>
       </geometry>
     </collision>
     <visual name='camera_visual'>
-      <origin xyz="0.2 0 0" rpy="0 0 0"/>
-      <geometry>
-        <box size="0.05 0.05 0.05"/>
+      <origin xyz="0.2 0 0" rpy="0 1.5707 0"/>
+      <geometry>
+        <cylinder radius="0.03" length="0.06"/>
+        <!-- <box size="0.05 0.05 0.05"/> -->
       </geometry>
       <!-- <material name="red"/> -->
@@ -173,5 +175,5 @@
   </link>
   <gazebo reference="camera">
-      <material>Gazebo/Orange</material>
+      <material>Gazebo/Black</material>
   </gazebo>
   <joint type="fixed" name="camera_joint">

Commit message: Make it into a Rumba :D

File: src/my_robot/urdf/my_robot.xacro (robot description, xacro)
@@ -34,18 +34,20 @@
     </inertial>
     <collision name='collision'>
-      <origin xyz="0 0 0" rpy=" 0 0 0"/>
-      <geometry>
-        <box size=".8 .4 .1"/>
+      <origin xyz="0 0 0" rpy="0 0 1.5707"/>
+      <geometry>
+        <cylinder radius="0.3" length="0.1"/>
+        <!-- <box size=".8 .4 .1"/> -->
       </geometry>
     </collision>
     <visual name='chassis_visual'>
-      <origin xyz="0 0 0" rpy=" 0 0 0"/>
-      <geometry>
-        <box size=".8 .4 .1"/>
+      <origin xyz="0 0 0" rpy="0 0 1.5707"/>
+      <geometry>
+        <cylinder radius="0.3" length="0.1"/>
+        <!-- <box size=".8 .4 .1"/> -->
       </geometry>
       <!-- <material name="blue"/> -->
     </visual>
     <collision name='back_caster_collision'>
-      <origin xyz="-0.3 0 -0.075" rpy=" 0 0 0"/>
+      <origin xyz="-0.2 0 -0.075" rpy=" 0 0 0"/>
       <geometry>
         <sphere radius="0.07499"/>
@@ -53,5 +55,5 @@
     </collision>
     <visual name='back_caster_visual'>
-      <origin xyz="-0.3 0 -0.075" rpy=" 0 0 0"/>
+      <origin xyz="-0.2 0 -0.075" rpy=" 0 0 0"/>
       <geometry>
         <sphere radius="0.075"/>
@@ -59,5 +61,5 @@
     </visual>
     <collision name='front_caster_collision'>
-      <origin xyz="0.3 0 -0.075" rpy=" 0 0 0"/>
+      <origin xyz="0.2 0 -0.075" rpy=" 0 0 0"/>
       <geometry>
         <sphere radius="0.07499"/>
@@ -65,5 +67,5 @@
     </collision>
     <visual name='front_caster_visual'>
-      <origin xyz="0.3 0 -0.075" rpy=" 0 0 0"/>
+      <origin xyz="0.2 0 -0.075" rpy=" 0 0 0"/>
       <geometry>
         <sphere radius="0.075"/>
@@ -150,5 +152,5 @@
     <inertial>
       <mass value="0.1"/>
-      <origin xyz="0.2 0 0" rpy="0 0 0"/>
+      <origin xyz="0.13 0 0" rpy="0 0 0"/>
       <inertia
           ixx="1e-6" ixy="0"   ixz="0"
@@ -159,5 +161,5 @@
     </inertial>
     <collision name='camera_collision'>
-      <origin xyz="0.2 0 0" rpy="0 1.5707 0"/>
+      <origin xyz="0.13 0 0" rpy="0 1.5707 0"/>
       <geometry>
         <!-- <box size="0.05 0.05 0.05"/> -->
@@ -166,5 +168,5 @@
     </collision>
     <visual name='camera_visual'>
-      <origin xyz="0.2 0 0" rpy="0 1.5707 0"/>
+      <origin xyz="0.13 0 0" rpy="0 1.5707 0"/>
       <geometry>
         <cylinder radius="0.03" length="0.06"/>

Commit message: Fix the hinges - so no translation is needed
to drive a robot
But it drives funny now :( Turns, stops etc

File: src/my_robot/urdf/my_robot.xacro (robot description, xacro)
@@ -144,5 +144,5 @@
     <child link="right_wheel"/>
     <parent link="chassis"/>
-    <axis xyz="0 -1 0" rpy="0 0 0"/>
+    <axis xyz="0 1 0" rpy="0 0 0"/>
     <limit effort="10000" velocity="1000"/>
     <dynamics damping="1.0" friction="1.0"/>

Commit message: Update my_robot with rtabmap and kinect

File: src/my_robot/urdf/my_robot.xacro (robot description, xacro)
@@ -176,5 +176,12 @@
     </visual>
   </link>
-  <gazebo reference="camera">
+  <joint name="camera_optical_joint" type="fixed">
+    <origin xyz="0 0 0" rpy="-1.5707 0 -1.5707"/>
+    <parent link="camera"/>
+    <child link="camera_link_optical"/>
+  </joint>
+  <link name="camera_link_optical">
+  </link>
+  <gazebo reference="camera_link_optical">
       <material>Gazebo/Black</material>
   </gazebo>

Commit message: Modify the camera so that it "sees well"

File: src/my_robot/urdf/my_robot.xacro (robot description, xacro)
@@ -152,5 +152,5 @@
     <inertial>
       <mass value="0.1"/>
-      <origin xyz="0.13 0 0" rpy="0 0 0"/>
+      <origin xyz="0.1 0 0" rpy="0 0 0"/>
       <inertia
           ixx="1e-6" ixy="0"   ixz="0"
@@ -161,14 +161,14 @@
     </inertial>
     <collision name='camera_collision'>
-      <origin xyz="0.13 0 0" rpy="0 1.5707 0"/>
+      <origin xyz="0.1 0 0" rpy="0 1.5707 0"/>
       <geometry>
         <!-- <box size="0.05 0.05 0.05"/> -->
-        <cylinder radius="0.03" length="0.06"/>
+        <cylinder radius="0.03" length="0.04"/>
       </geometry>
     </collision>
     <visual name='camera_visual'>
-      <origin xyz="0.13 0 0" rpy="0 1.5707 0"/>
-      <geometry>
-        <cylinder radius="0.03" length="0.06"/>
+      <origin xyz="0.1 0 0" rpy="0 1.5707 0"/>
+      <geometry>
+        <cylinder radius="0.03" length="0.04"/>
         <!-- <box size="0.05 0.05 0.05"/> -->
       </geometry>
